Commit message: Robot can run with teleop twist keyboard

File: diff_bot_description/description/base.xacro (robot description, xacro)
@@ -3,35 +3,26 @@
   <!-- Variables -->
   <xacro:property name="base_length" value="0.498"/>
-  <xacro:property name="base_width" value="0.4"/>
-  <xacro:property name="base_height" value="0.02"/>
-  <xacro:property name="top_length" value="0.246"/>
-  <xacro:property name="top_width" value="0.361"/>
-  <xacro:property name="top_height" value="0.03"/>
-  <xacro:property name="clearance" value="0.05"/>
+  <xacro:property name="base_width" value="0.39"/>
+  <xacro:property name="base_height" value="0.04"/>
+  <xacro:include filename="inertial_macros.xacro"/>
   <!-- Base Link -->
   <link name="base_link"/>
-  <!-- Base Plate -->
+  <!-- Chassis -->
   <joint name="base_joint" type="fixed">
-    <origin xyz="0.0 0.0 ${clearance + base_height + 0.01}"/>  <!-- 1cm provided for no clipping -->
+    <origin xyz="0.0 0.0 0.0"/>
     <parent link="base_link"/>
-    <child link="base_plate"/>
+    <child link="chassis"/>
   </joint>
-  <link name="base_plate">
-    <inertial>
-      <origin xyz="0.0 0.0 -${base_height/2}"/>
-      <mass value="0.0"/>
-      <inertia ixx="0.0" ixy="0.0" ixz="0.0" iyy="0.0" iyz="0.0" izz="0.0"/>
-    </inertial>
+  <link name="chassis">
     <visual>
-      <origin xyz="0.0 0.0 -${base_height/2}"/>
+      <origin xyz="-0.019 0.0 0.0115"/>
       <geometry>
-        <box size="${base_length} ${base_width} ${base_height}"/>
+        <mesh filename="${mesh_path}/chassis.stl"/>
+        <!-- <mesh filename="/home/subham/ros_ws/diff_drive/src/diff_bot_description/meshes/chassis.stl" scale="1 1 1"/> -->
       </geometry>
-      <material name="blue">
-        <color rgba="0.0 0.0 1.0 1.0"/>
-      </material>
+      <material name="blue"></material>
     </visual>
     <collision>
-      <origin xyz="0.0 0.0 -${base_height/2}"/>
+      <origin xyz="0.229 0.0 0.0315"/>
       <geometry>
         <box size="${base_length} ${base_width} ${base_height}"/>
@@ -39,35 +30,6 @@
     </collision>
     <xacro:inertial_box mass="1.0" x="${base_length}" y="${base_width}" z="${base_height}">
-      <origin xyz="0.0 0.0 -${base_height/2}"/>
+      <origin xyz="0.0 0.0 0.0"/>
     </xacro:inertial_box>
   </link>
-  <!-- Top Plate -->
-  <!-- <joint name="top_joint" type="fixed">
-    <origin xyz="-${base_length/2 - top_length/2} ${base_width/2 - top_width/2} ${top_height}"/>
-    <parent link="base_plate"/>
-    <child link="top_plate"/>
-  </joint>
-  <link name="top_plate">
-    <inertial>
-      <origin xyz="0.0 0.0 -${top_height/2}"/>
-      <mass value="0.0"/>
-      <inertia ixx="0.0" ixy="0.0" ixz="0.0" iyy="0.0" iyz="0.0" izz="0.0"/>
-    </inertial>
-    <visual name="">
-      <origin xyz="0.0 0.0 -${top_height/2}"/>
-      <geometry>
-        <box size="${top_length} ${top_width} ${top_height}"/>
-      </geometry>
-      <material name="blue">
-        <color rgba="0.0 0.0 1.0 1.0"/>
-        <texture filename=""/>
-      </material>
-    </visual>
-    <collision>
-      <origin xyz="0.0 0.0 -${top_height/2}"/>
-      <geometry>
-        <box size="${top_length} ${top_width} ${top_height}"/>
-      </geometry>
-    </collision>
-  </link> -->
 </robot>

File: diff_bot_description/description/bot.urdf.xacro (robot description, xacro)
@@ -1,15 +1,22 @@
 <?xml version="1.0"?>
-<robot xmlns:xacro="http://www.ros.org/wiki/xacro"  name="Diff_Bot">
-    <!-- Base Plate -->
+<robot xmlns:xacro="http://www.ros.org/wiki/xacro"  name="diff_bot">
+    <!-- Inertial Macros -->
     <xacro:include filename="inertial_macros.xacro"/>
-    <!-- Base Plate -->
+    <!-- Materials -->
+    <xacro:include filename="materials.xacro"/>
+    <!-- Gazebo plugins -->
+    <xacro:include filename="gazebo.xacro"/>
+    <!-- Mesh/STL files Path -->
+    <xacro:property name="mesh_path"
+    value="file:///home/subham/ros_ws/diff_drive/src/diff_bot_description/meshes"/>
+    <!-- Chassis -->
     <xacro:include filename="base.xacro"/>
-    <!-- Caster -->
+    <!-- Rear Wheels -->
+    <xacro:include filename="wheels.xacro"/>
+    <!-- Caster Wheels -->
     <xacro:include filename="caster.xacro"/>
-    <!-- Wheels -->
-    <xacro:include filename="wheels.xacro"/>
     <!-- LIDAR -->
     <xacro:include filename="lidar.xacro"/>
-    <!-- ROS Control -->
-    <!-- <xacro:include filename="ros2_control.xacro"/> -->
+    <!-- ROS2 Control -->
+    <xacro:include filename="ros2_control.xacro"/>
 </robot>

File: diff_bot_description/description/caster.xacro (robot description, xacro)
@@ -2,6 +2,6 @@
 <robot xmlns:xacro="http://www.ros.org/wiki/xacro">
     <!-- Variables -->
-    <xacro:property name="caster_radius" value="0.02" />
-    <xacro:property name="caster_gap" value="0.046" />
+    <xacro:property name="caster_radius" value="0.021" />
+    <xacro:property name="caster_gap" value="0.021" />
     <!-- Caster Macro (sphere) -->
     <xacro:macro name="caster" params="prefix parent x y z z_sign">
@@ -13,5 +13,5 @@
         </joint>
         <link name="${prefix}_caster">
-            <visual>
+            <!-- <visual>
                 <geometry>
                     <sphere radius="${caster_radius}"/>
@@ -20,5 +20,5 @@
                     <color rgba="0 0 0 1"/>
                 </material>
-            </visual>
+            </visual> -->
             <collision>
                 <geometry>
@@ -27,10 +27,10 @@
             </collision>
             <xacro:inertial_sphere mass="0.1" radius="${caster_radius}">
-             <origin xyz="0 0 0"/>
+                <origin xyz="0 0 0"/>
             </xacro:inertial_sphere>
         </link>
     </xacro:macro>
     <!-- Casters (two at the bottom) -->
-    <xacro:caster prefix="top_left" parent="base_plate" x="${base_length/2 - 0.01}" y="${base_width/2 - 0.01 }" z="${-caster_gap}" z_sign="-1"/>
-    <xacro:caster prefix="top_right" parent="base_plate" x="${base_length/2 - 0.01}" y="-${base_width/2 - 0.01 }" z="${-caster_gap}" z_sign="1"/>
+    <xacro:caster prefix="top_left" parent="chassis" x="0.45" y="0.185" z="${-caster_gap}" z_sign="-1"/>
+    <xacro:caster prefix="top_right" parent="chassis" x="0.45" y="-0.185" z="${-caster_gap}" z_sign="1"/>
 </robot>

File: diff_bot_description/description/lidar.xacro (robot description, xacro)
@@ -6,20 +6,19 @@
   <!-- Links -->
   <joint name="lidar_joint" type="fixed">
-    <origin xyz="0 0 ${lidar_height/2}"/>
-    <parent link="base_plate"/>
+    <origin xyz="0.4875 0.0 0.06"/>
+    <parent link="chassis"/>
     <child link="lidar_link"/>
   </joint>
   <link name="lidar_link">
     <visual>
-      <origin xyz="0 0 0"/>
+      <origin xyz="0 0 -0.08"/>
       <geometry>
-        <cylinder length="${lidar_height}" radius="${lidar_radius}"/>
+        <mesh filename="${mesh_path}/lidar.stl"/>
+        <!-- <mesh filename="/home/subham/ros_ws/diff_drive/src/diff_bot_description/meshes/lidar.stl" scale="1 1 1"/> -->
       </geometry>
-      <material name="red">
-        <color rgba="1 0 0 1"/>
-      </material>
+      <material name="red"/>
     </visual>
     <collision>
-      <origin xyz="0 0 0"/>
+      <origin xyz="0 0 0.05"/>
       <geometry>
         <cylinder length="${lidar_height}" radius="${lidar_radius}"/>
@@ -30,42 +29,3 @@
     </xacro:inertial_cylinder>
   </link>
-  <gazebo reference="lidar_link">
-    <material>Gazebo/Red</material>
-    <sensor type="ray" name="lidar_sensor">
-      <pose>0 0 0 0 0 0</pose>
-      <visualize>true</visualize>
-      <update_rate>10</update_rate>
-      <ray>
-        <scan>
-          <horizontal>
-            <samples>360</samples>
-            <resolution>1</resolution>
-            <min_angle>-${pi}</min_angle>
-            <max_angle>${pi}</max_angle>
-          </horizontal>
-          <range>
-            <min>0.12</min>
-            <max>6</max>
-          </range>
-        </scan>
-        <range>
-          <min>0.3</min>
-          <max>12</max>
-          <resolution>0.01</resolution>
-        </range>
-        <noise>
-          <type>gaussian</type>
-          <mean>0.0</mean>
-          <stddev>0.01</stddev>
-        </noise>
-      </ray>
-      <plugin name="gazebo_ros_lidar" filename="libgazebo_ros_ray_sensor.so">
-        <ros>
-          <argument> ~/out:=scan </argument>
-        </ros>
-        <output_type>sensor_msgs/LaserScan</output_type>
-        <frame_name>lidar_link</frame_name>
-      </plugin>
-    </sensor>
-  </gazebo>
 </robot>

File: diff_bot_description/description/ros2_control.xacro (robot description, xacro)
@@ -1,62 +1,58 @@
 <?xml version="1.0"?>
 <robot xmlns:xacro="http://www.ros.org/wiki/xacro">
-    <!-- <xacro:unless value="$(arg sim_mode)"> -->
-        <ros2_control name="RealRobot" type="system">
-            <hardware>
-                <plugin>diffdrive_arduino/DiffDriveArduino</plugin>
-                <param name="left_wheel_name">bottom_left_joint</param>
-                <param name="right_wheel_name">bottom_right_joint</param>
-                <param name="loop_rate">30</param>
-                <param name="device">/dev/ttyACM0</param>
-                <param name="baud_rate">57600</param>
-                <param name="timeout">1000</param>
-                <param name="enc_counts_per_rev">559</param>
-            </hardware>
-            <joint name="bottom_left_joint">
-                <command_interface name="velocity">
-                    <param name="min">-10</param>
-                    <param name="max">10</param>
-                </command_interface>
-                <state_interface name="velocity"/>
-                <state_interface name="position"/>
-            </joint>
-            <joint name="bottom_right_joint">
-                <command_interface name="velocity">
-                    <param name="min">-10</param>
-                    <param name="max">10</param>
-                </command_interface>
-                <state_interface name="velocity"/>
-                <state_interface name="position"/>
-            </joint>
-        </ros2_control>
-    <!-- </xacro:unless> -->
-    <!-- <xacro:if value="$(arg sim_mode)">
-        <ros2_control name="GazeboSystem" type="system">
-            <hardware>
-                <plugin>gazebo_ros2_control/GazeboSystem</plugin>
-            </hardware>
-            <joint name="left_wheel_joint">
-                <command_interface name="velocity">
-                    <param name="min">-10</param>
-                    <param name="max">10</param>
-                </command_interface>
-                <state_interface name="velocity"/>
-                <state_interface name="position"/>
-            </joint>
-            <joint name="right_wheel_joint">
-                <command_interface name="velocity">
-                    <param name="min">-10</param>
-                    <param name="max">10</param>
-                </command_interface>
-                <state_interface name="velocity"/>
-                <state_interface name="position"/>
-            </joint>
-        </ros2_control>
-    </xacro:if> -->
+    <ros2_control name="GazeboSimSystem" type="system">
+        <hardware>
+            <plugin>gz_ros2_control/GazeboSimSystem</plugin>
+        </hardware>
+        <joint name="bottom_left_wheel_joint">
+            <command_interface name="velocity">
+                <param name="min">-10</param>
+                <param name="max">10</param>
+            </command_interface>
+            <state_interface name="position"/>
+            <state_interface name="velocity"/>
+        </joint>
+        <joint name="bottom_right_wheel_joint">
+            <command_interface name="velocity">
+                <param name="min">-10</param>
+                <param name="max">10</param>
+            </command_interface>
+            <state_interface name="position"/>
+            <state_interface name="velocity"/>
+        </joint>
+    </ros2_control>
     <!-- <gazebo>
-        <plugin name="gazebo_ros2_control" filename="libgazebo_ros2_control.so">
-            <parameters>$(find articubot_one)/config/my_controllers.yaml</parameters>
-            <parameters>$(find articubot_one)/config/gaz_ros2_ctl_use_sim.yaml</parameters>
+        <plugin filename="gz_ros2_control-system.so"
+                name="gz_ros2_control::GazeboSimROS2ControlPlugin">
+            <parameters>/home/subham/ros_ws/diff_drive/install/diff_bot_description/share/diff_bot_description/config/controllers.yaml</parameters>
         </plugin>
     </gazebo> -->
+    <!-- <ros2_control name="RealRobot" type="system">
+        <hardware>
+            <plugin>diffdrive_arduino/DiffDriveArduino</plugin>
+            <param name="left_wheel_name">bottom_left_joint</param>
+            <param name="right_wheel_name">bottom_right_joint</param>
+            <param name="loop_rate">30</param>
+            <param name="device">/dev/ttyACM0</param>
+            <param name="baud_rate">57600</param>
+            <param name="timeout">1000</param>
+            <param name="enc_counts_per_rev">559</param>
+        </hardware>
+        <joint name="bottom_left_joint">
+            <command_interface name="velocity">
+                <param name="min">-10</param>
+                <param name="max">10</param>
+            </command_interface>
+            <state_interface name="velocity"/>
+            <state_interface name="position"/>
+        </joint>
+        <joint name="bottom_right_joint">
+            <command_interface name="velocity">
+                <param name="min">-10</param>
+                <param name="max">10</param>
+            </command_interface>
+            <state_interface name="velocity"/>
+            <state_interface name="position"/>
+        </joint>
+    </ros2_control> -->
 </robot>

File: diff_bot_description/description/wheels.xacro (robot description, xacro)
@@ -2,27 +2,28 @@
 <robot xmlns:xacro="http://www.ros.org/wiki/xacro">
   <!-- Variables -->
-  <xacro:property name="wheel_radius" value="0.035" />
+  <xacro:property name="wheel_radius" value="0.0425" />
   <xacro:property name="wheel_width" value="0.04" />
   <xacro:property name="wheel_gap" value="0.009" />
   <!-- Wheel Macro -->
-  <xacro:macro name="wheel" params="prefix parent x y z z_sign">
-    <joint name="${prefix}_joint" type="continuous">
+  <xacro:macro name="wheel" params="prefix parent x y z rotation">
+    <joint name="${prefix}_wheel_joint" type="continuous">
       <parent link="${parent}"></parent>
       <child link="${prefix}_wheel"></child>
-      <origin xyz="${x} ${y} ${z}" rpy="${z_sign * pi/2} 0 0" />
-      <axis xyz="0 0 ${-1 * z_sign}" />
+      <origin xyz="${x} ${y} ${z}" rpy="${rotation * pi/2} 0 0" />
+      <axis xyz="0 0 ${rotation * -1}" />
     </joint>
     <link name="${prefix}_wheel">
       <visual>
+        <origin xyz="0 0 0" rpy="${pi/2} 0 0"/>
         <geometry>
-          <cylinder radius="${wheel_radius}" length="${wheel_width}"/>
+          <mesh filename="${mesh_path}/wheel.stl"/>
+          <!-- <mesh filename="/home/subham/ros_ws/diff_drive/src/diff_bot_description/meshes/wheel.stl" scale="1 1 1"/> -->
         </geometry>
-        <material name="black">
-          <color rgba="0 0 0 1"/>
-        </material>
+        <material name="black"/>
       </visual>
       <collision>
+        <origin xyz="0 0 -0.02"/>
         <geometry>
-          <cylinder radius="${wheel_radius}" length="${wheel_width}"/>
+           <sphere radius="${wheel_radius}"/>
         </geometry>
       </collision>
@@ -33,7 +34,5 @@
   </xacro:macro>
   <!-- Wheels -->
-  <!-- <xacro:wheel prefix="top_left" parent="base_plate" x="${base_width/2 - 0.03}" y="${base_length/2 + wheel_gap + wheel_width/2}" z="-0.04" z_sign="1"/>
-  <xacro:wheel prefix="top_right" parent="base_plate" x="${base_width/2 - 0.03}" y="-${base_length/2 + wheel_gap + wheel_width/2}" z="-0.04" z_sign="1"/> -->
-  <xacro:wheel prefix="bottom_left" parent="base_plate" x="-${base_length/2 - 0.013}" y="${base_width/2 + wheel_gap + wheel_width/2}" z="-0.04" z_sign="-1"/>
-  <xacro:wheel prefix="bottom_right" parent="base_plate" x="-${base_length/2 - 0.013}" y="-${base_width/2 + wheel_gap + wheel_width/2}" z="-0.04" z_sign="1"/>
+  <xacro:wheel prefix="bottom_left" parent="chassis" x="0.0" y="0.21" z="0.0" rotation="1"/>
+  <xacro:wheel prefix="bottom_right" parent="chassis" x="0.0" y="-0.21" z="0.0" rotation="-1"/>
 </robot>
